File: hardware/esp32c3-radio-adapter/esp32c3-radio-adapter.kicad_sch (KiCad schematic)
At the start: 10 parts, among them J1 Conn_01x08, J2 Conn_01x08, J3 E07-M1101D_or_Ra-02, J4 Expansion

Commit message: Adapters: reassign the GPIOs so the socket adapter routes on one layer
The pin-header (socket) adapter is now entirely on the back copper, the
expansion header and strap included; the front carries only pads and the
GND pour.  New assignment, shared by both adapters:

  MOSI GPIO8, SCK GPIO9, CSN/NSS GPIO0, MISO GPIO7, GDO0/RST(DIO0) GPIO10,
  GDO2/DIO0(DIO1) GPIO6, strap RADIO_ID GPIO5, SX1278 module RESET GPIO4.

GPIO8/9 are boot strapping pins but carry only ESP32 outputs, which float
at boot; the radio's outputs stay on plain GPIOs.  On the socket adapter
the radio signals then all leave the GPIO row, which faces the socket, in
the order its pads want them: GDO0 and SCK drop straight in, MOSI and MISO
via one lane each, GDO2 round the left of the socket into its pad from
below.  CSN/NSS (GPIO0, the last power-row pin) passes under its own pad,
crosses between the rows (now otherwise empty) and drops through a
GPIO-row gap.  GND and 3V3 leave the power row upward, run along the top
edge above the header and down the strip right of the SuperMini into the
socket's right column; GND continues under the socket to the strap.

Expansion header J4 (centred): 3V3, GPIO4, 3, 2, 1, 21, 20 - GPIO4..1 rise
straight up, GPIO21/20 come up the right-hand strip.  5V is dropped: its
pad sits under the top-left hole and cannot be reached on one layer.  The
strap moves to the bottom-left corner (JP1 header, R1 0805 on the back),
fed by GPIO5 dropping straight down and by the under-socket GND lane.

SX1278 module adapter: same map; its GPIO order matches the module's pad
order so the front-copper lanes stay nested; NSS and RESET now come from
the right column on the back copper, 3V3 goes down the right of the
SuperMini, and GPIO5 is tied to 3V3 across the top.

Both adapters pass ERC and DRC; the antenna keepout starts 1.6 mm inboard
of the power row (was 1.3) to give CSN/NSS its lane under the last pad.

Co-Authored-By: Claude Fable 5.1 <noreply@anthropic.com>
Claude-Session: https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
Parts:
- R1: footprint Adapter:R_0805_2012Metric_HandSolder_AlongY -> Adapter:R_0805_2012Metric_HandSolder_AlongY_Back
Connections:
- net +3V3: now also J4.1 (Pin_1)
- net +5V: no longer J4.1 (Pin_1)
- net CSN_NSS: now also J2.8 (Pin_8); no longer J1.3 (Pin_3)
- net GDO2_DIO0: now also J1.2 (Pin_2); no longer J2.5 (Pin_5)
- net GPIO20: now also J4.7 (Pin_7); no longer J4.5 (Pin_5)
- net GPIO21: now also J4.6 (Pin_6); no longer J4.7 (Pin_7)
- net MISO: now also J1.3 (Pin_3); no longer J2.4 (Pin_4)
- net MOSI: now also J1.4 (Pin_4); no longer J1.1 (Pin_1)
- net RADIO_ID: now also J1.1 (Pin_1); no longer J2.7 (Pin_7)
- net SCK: now also J1.5 (Pin_5); no longer J1.2 (Pin_2)
- removed net GPIO0: J2.8 (Pin_8), J4.6 (Pin_6)
- net GPIO8 renamed GPIO4
- net GPIO4: now also J2.4 (Pin_4); no longer J1.4 (Pin_4)
- net GPIO9 renamed GPIO3
- net GPIO3: now also J2.5 (Pin_5); no longer J1.5 (Pin_5)
- new net GPIO1: J2.7 (Pin_7), J4.5 (Pin_5)
Other:
- note added: "ESP32-C3 SuperMini (J1 = GPIO row, J2 = power row; through-hole or castellated) driving a CC1101 E07-M1101D board or an SX1278 Ra-02 breakout in socket J3. SPI: MOSI=GPIO8 SCK=GPIO9 CSN/NSS=GPIO0 MISO=GPIO7; GDO0 (Ra-02: RST)=GPIO10, GDO2 (Ra-02: DIO0)=GPIO6. J4: 3V3 and the unused GPIOs. JP1 (jumper) or R1 (0R): radio-type strap on GPIO5 (RADIO_ID) to GND, open = CC1101, fitted = Ra-02. H1-H4: M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"
- note removed: "ESP32-C3 SuperMini (J1 = GPIO row, J2 = power row; through-hole or castellated) driving a CC1101 E07-M1101D board or an SX1278 Ra-02 breakout in socket J3. SPI: MOSI=GPIO5 SCK=GPIO6 CSN/NSS=GPIO7 MISO=GPIO4; GDO0 (Ra-02: RST)=GPIO10, GDO2 (Ra-02: DIO0)=GPIO3. J4: the unused SuperMini pins. JP1 (jumper) or R1 (0R): radio-type strap on GPIO1 (RADIO_ID) to GND, open = CC1101, fitted = Ra-02. H1-H4: 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"
Changed lines of the file:
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@@
 		(title "ESP32-C3 SuperMini to CC1101 (E07-M1101D) or SX1278 Ra-02 breakout adapter")
 		(rev "${GIT_DESCRIBE}")
-		(comment 1 "Carrier joining an ESP32-C3 SuperMini to an Ebyte E07-M1101D-SMA CC1101 board or an SX1278 Ra-02 breakout via one 2x4 socket; radio tracks on the back, GND pour plus the expansion header and strap on the front")
+		(comment 1 "Carrier joining an ESP32-C3 SuperMini to an Ebyte E07-M1101D-SMA CC1101 board or an SX1278 Ra-02 breakout via one 2x4 socket; all tracks on the back, GND pour on the front")
 	)
 	(symbol
@@
 		)
 	)
+	(global_label "RADIO_ID"
+		(shape bidirectional)
+		(at 71.12 93.98 180)
+		(fields_autoplaced yes)
+		(effects
+			(font
+				(size 1.27 1.27)
+			)
+			(justify right)
+		)
+		(property "Intersheetrefs" "${INTERSHEET_REFS}"
+			(at 71.12 93.98 0)
+			(effects
+				(font
+					(size 1.27 1.27)
+				)
+				(justify right)
+				(hide yes)
+			)
+		)
+	)
+	(global_label "GDO2_DIO0"
+		(shape bidirectional)
+		(at 71.12 96.52 180)
+		(fields_autoplaced yes)
+		(effects
+			(font
+				(size 1.27 1.27)
+			)
+			(justify right)
+		)
+		(property "Intersheetrefs" "${INTERSHEET_REFS}"
+			(at 71.12 96.52 0)
+			(effects
+				(font
+					(size 1.27 1.27)
+				)
+				(justify right)
+				(hide yes)
+			)
+		)
+	)
+	(global_label "MISO"
+		(shape bidirectional)
+		(at 71.12 99.06 180)
+		(fields_autoplaced yes)
+		(effects
+			(font
+				(size 1.27 1.27)
+			)
+			(justify right)
+		)
+		(property "Intersheetrefs" "${INTERSHEET_REFS}"
+			(at 71.12 99.06 0)
+			(effects
+				(font
+					(size 1.27 1.27)
+				)
+				(justify right)
+				(hide yes)
+			)
+		)
+	)
 	(global_label "MOSI"
 		(shape bidirectional)
-		(at 71.12 93.98 180)
-		(fields_autoplaced yes)
-		(effects
-			(font
-				(size 1.27 1.27)
-			)
-			(justify right)
-		)
-		(property "Intersheetrefs" "${INTERSHEET_REFS}"
-			(at 71.12 93.98 0)
+		(at 71.12 101.6 180)
+		(fields_autoplaced yes)
+		(effects
+			(font
+				(size 1.27 1.27)
+			)
+			(justify right)
+		)
+		(property "Intersheetrefs" "${INTERSHEET_REFS}"
+			(at 71.12 101.6 0)
 			(effects
 				(font
@@
 	)
 	(global_label "SCK"
-		(shape bidirectional)
-		(at 71.12 96.52 180)
-		(fields_autoplaced yes)
-		(effects
-			(font
-				(size 1.27 1.27)
-			)
-			(justify right)
-		)
-		(property "Intersheetrefs" "${INTERSHEET_REFS}"
-			(at 71.12 96.52 0)
-			(effects
-				(font
-					(size 1.27 1.27)
-				)
-				(justify right)
-				(hide yes)
-			)
-		)
-	)
-	(global_label "CSN_NSS"
-		(shape bidirectional)
-		(at 71.12 99.06 180)
-		(fields_autoplaced yes)
-		(effects
-			(font
-				(size 1.27 1.27)
-			)
-			(justify right)
-		)
-		(property "Intersheetrefs" "${INTERSHEET_REFS}"
-			(at 71.12 99.06 0)
-			(effects
-				(font
-					(size 1.27 1.27)
-				)
-				(justify right)
-				(hide yes)
-			)
-		)
-	)
-	(global_label "GPIO8"
-		(shape bidirectional)
-		(at 71.12 101.6 180)
-		(fields_autoplaced yes)
-		(effects
-			(font
-				(size 1.27 1.27)
-			)
-			(justify right)
-		)
-		(property "Intersheetrefs" "${INTERSHEET_REFS}"
-			(at 71.12 101.6 0)
-			(effects
-				(font
-					(size 1.27 1.27)
-				)
-				(justify right)
-				(hide yes)
-			)
-		)
-	)
-	(global_label "GPIO9"
 		(shape bidirectional)
 		(at 71.12 104.14 180)
@@
 		)
 	)
-	(global_label "MISO"
+	(global_label "GPIO4"
 		(shape bidirectional)
 		(at 96.52 101.6 180)
@@
 		)
 	)
-	(global_label "GDO2_DIO0"
+	(global_label "GPIO3"
 		(shape bidirectional)
 		(at 96.52 104.14 180)
@@
 		)
 	)
-	(global_label "RADIO_ID"
+	(global_label "GPIO1"
 		(shape bidirectional)
 		(at 96.52 109.22 180)
@@
 		)
 	)
-	(global_label "GPIO0"
+	(global_label "CSN_NSS"
 		(shape bidirectional)
 		(at 96.52 111.76 180)
@@
 		)
 	)
-	(global_label "+5V"
+	(global_label "+3V3"
 		(shape bidirectional)
 		(at 147.32 119.38 180)
@@
 		)
 	)
-	(global_label "GPIO8"
+	(global_label "GPIO4"
 		(shape bidirectional)
 		(at 147.32 121.92 180)
@@
 		)
 	)
-	(global_label "GPIO9"
+	(global_label "GPIO3"
 		(shape bidirectional)
 		(at 147.32 124.46 180)
@@
 		)
 	)
+	(global_label "GPIO1"
+		(shape bidirectional)
+		(at 147.32 129.54 180)
+		(fields_autoplaced yes)
+		(effects
+			(font
+				(size 1.27 1.27)
+			)
+			(justify right)
+		)
+		(property "Intersheetrefs" "${INTERSHEET_REFS}"
+			(at 147.32 129.54 0)
+			(effects
+				(font
+					(size 1.27 1.27)
+				)
+				(justify right)
+				(hide yes)
+			)
+		)
+	)
+	(global_label "GPIO21"
+		(shape bidirectional)
+		(at 147.32 132.08 180)
+		(fields_autoplaced yes)
+		(effects
+			(font
+				(size 1.27 1.27)
+			)
+			(justify right)
+		)
+		(property "Intersheetrefs" "${INTERSHEET_REFS}"
+			(at 147.32 132.08 0)
+			(effects
+				(font
+					(size 1.27 1.27)
+				)
+				(justify right)
+				(hide yes)
+			)
+		)
+	)
 	(global_label "GPIO20"
-		(shape bidirectional)
-		(at 147.32 129.54 180)
-		(fields_autoplaced yes)
-		(effects
-			(font
-				(size 1.27 1.27)
-			)
-			(justify right)
-		)
-		(property "Intersheetrefs" "${INTERSHEET_REFS}"
-			(at 147.32 129.54 0)
-			(effects
-				(font
-					(size 1.27 1.27)
-				)
-				(justify right)
-				(hide yes)
-			)
-		)
-	)
-	(global_label "GPIO0"
-		(shape bidirectional)
-		(at 147.32 132.08 180)
-		(fields_autoplaced yes)
-		(effects
-			(font
-				(size 1.27 1.27)
-			)
-			(justify right)
-		)
-		(property "Intersheetrefs" "${INTERSHEET_REFS}"
-			(at 147.32 132.08 0)
-			(effects
-				(font
-					(size 1.27 1.27)
-				)
-				(justify right)
-				(hide yes)
-			)
-		)
-	)
-	(global_label "GPIO21"
 		(shape bidirectional)
 		(at 147.32 134.62 180)
@@
 			)
 		)
-		(property "Footprint" "Adapter:R_0805_2012Metric_HandSolder_AlongY"
+		(property "Footprint" "Adapter:R_0805_2012Metric_HandSolder_AlongY_Back"
 			(at 203.2 127 0)
 			(effects
@@
 		)
 	)
-	(text "ESP32-C3 SuperMini (J1 = GPIO row, J2 = power row; through-hole or castellated) driving a CC1101 E07-M1101D board or an SX1278 Ra-02 breakout in socket J3.\nSPI: MOSI=GPIO5 SCK=GPIO6 CSN/NSS=GPIO7 MISO=GPIO4; GDO0 (Ra-02: RST)=GPIO10, GDO2 (Ra-02: DIO0)=GPIO3.\nJ4: the unused SuperMini pins.  JP1 (jumper) or R1 (0R): radio-type strap on GPIO1 (RADIO_ID) to GND, open = CC1101, fitted = Ra-02.\nH1-H4: M2 mounting holes.  Radio tracks on B.Cu; F.Cu carries the GND pour, J4's tracks and the strap."
+	(text "ESP32-C3 SuperMini (J1 = GPIO row, J2 = power row; through-hole or castellated) driving a CC1101 E07-M1101D board or an SX1278 Ra-02 breakout in socket J3.\nSPI: MOSI=GPIO8 SCK=GPIO9 CSN/NSS=GPIO0 MISO=GPIO7; GDO0 (Ra-02: RST)=GPIO10, GDO2 (Ra-02: DIO0)=GPIO6.\nJ4: 3V3 and the unused GPIOs.  JP1 (jumper) or R1 (0R): radio-type strap on GPIO5 (RADIO_ID) to GND, open = CC1101, fitted = Ra-02.\nH1-H4: M2 mounting holes.  All tracks on B.Cu; F.Cu carries only a GND pour."
 		(exclude_from_sim no)
 		(at 60 90 0)
