File: hardware/esp32c3-sx1278-adapter/esp32c3-sx1278-adapter.kicad_pcb (KiCad board)
At the start: 2 copper layers, 24 x 58 mm, 5 parts, among them J1 Conn_01x08, J2 Conn_01x08, J3 Antenna, J4 SMA, U2 SX1278_module

Commit message: SX1278 module adapter: move NSS and RESET off the GPIO8/GPIO9 straps
Same boot-strap hazard as the socket adapter: the module's NSS sat on GPIO9
(the BOOT strap) and RESET on GPIO8, so at reset the module's pin capacitance
could hold a strap low through the weak internal pull-up and drop the chip
into USB download mode.  On this two-layer board the fix keeps the nested
front-copper left bus by shifting the chain: NSS GPIO9 -> GPIO10, DIO0
GPIO10 -> GPIO20, RESET GPIO8 -> GPIO21, so the pad order still matches the
pin order and no lane crosses.  GPIO8 and GPIO9 are now unused.  The old
bottom-copper RESET run is removed.  README and schematic note updated;
ERC/DRC clean.

Co-Authored-By: Claude Opus 4.8 <noreply@anthropic.com>
Claude-Session: https://claude.ai/code/session_01JoGdh4Cg3VtTTDZi4gQuiN
Connections:
- J1 pad 4: RESET -> GPIO8
- J1 pad 5: NSS -> GPIO9
- J1 pad 6: DIO0 -> NSS
- J1 pad 7: GPIO20 -> DIO0
- J1 pad 8: GPIO21 -> RESET
Routing:
- net RESET: track 22.7 -> 12.6 mm, vias 1 -> 0
- net NSS: track 22.7 -> 20.2 mm
- net DIO0: track 18.9 -> 16.4 mm
Changed lines of the file:
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@@
 	(net 2 "DIO1")
 	(net 3 "MISO")
-	(net 4 "RESET")
-	(net 5 "NSS")
-	(net 6 "DIO0")
-	(net 7 "GPIO20")
-	(net 8 "GPIO21")
+	(net 4 "GPIO8")
+	(net 5 "GPIO9")
+	(net 6 "NSS")
+	(net 7 "DIO0")
+	(net 8 "RESET")
 	(net 9 "+5V")
 	(net 10 "GND")
@@
 			(layers "*.Cu" "*.Mask")
 			(remove_unused_layers no)
-			(net 4 "RESET")
+			(net 4 "GPIO8")
 			(pinfunction "Pin_4")
 			(pintype "passive")
@@
 			(layers "*.Cu" "*.Mask")
 			(remove_unused_layers no)
-			(net 5 "NSS")
+			(net 5 "GPIO9")
 			(pinfunction "Pin_5")
 			(pintype "passive")
@@
 			(layers "*.Cu" "*.Mask")
 			(remove_unused_layers no)
-			(net 6 "DIO0")
+			(net 6 "NSS")
 			(pinfunction "Pin_6")
 			(pintype "passive")
@@
 			(layers "*.Cu" "*.Mask")
 			(remove_unused_layers no)
-			(net 7 "GPIO20")
+			(net 7 "DIO0")
 			(pinfunction "Pin_7")
 			(pintype "passive")
@@
 			(layers "*.Cu" "*.Mask")
 			(remove_unused_layers no)
-			(net 8 "GPIO21")
+			(net 8 "RESET")
 			(pinfunction "Pin_8")
 			(pintype "passive")
@@
 			(size 1 3)
 			(layers "F.Cu" "F.Mask" "F.Paste")
-			(net 5 "NSS")
+			(net 6 "NSS")
 			(pinfunction "Pin_9")
 			(pintype "passive")
@@
 			(size 1 3)
 			(layers "F.Cu" "F.Mask" "F.Paste")
-			(net 6 "DIO0")
+			(net 7 "DIO0")
 			(pinfunction "Pin_10")
 			(pintype "passive")
@@
 			(size 1 3)
 			(layers "F.Cu" "F.Mask" "F.Paste")
-			(net 4 "RESET")
+			(net 8 "RESET")
 			(pinfunction "Pin_11")
 			(pintype "passive")
@@
 		)
 	)
-	(gr_text "RESET"
-		(at 105.2 111.62 0)
-		(layer "F.SilkS")
-		(effects
-			(font
-				(size 0.6 0.6)
-				(thickness 0.09)
-			)
-			(justify left)
-		)
-	)
 	(gr_text "9"
 		(at 102.8 114.16 0)
@@
 		)
 	)
-	(gr_text "NSS"
-		(at 105.2 114.16 0)
-		(layer "F.SilkS")
-		(effects
-			(font
-				(size 0.6 0.6)
-				(thickness 0.09)
-			)
-			(justify left)
-		)
-	)
 	(gr_text "10"
 		(at 102.8 116.7 0)
@@
 		)
 	)
-	(gr_text "DIO0"
+	(gr_text "NSS"
 		(at 105.2 116.7 0)
 		(layer "F.SilkS")
@@
 		)
 	)
+	(gr_text "DIO0"
+		(at 105.2 119.24 0)
+		(layer "F.SilkS")
+		(effects
+			(font
+				(size 0.6 0.6)
+				(thickness 0.09)
+			)
+			(justify left)
+		)
+	)
 	(gr_text "21"
 		(at 102.8 121.78 0)
@@
 		)
 	)
+	(gr_text "RESET"
+		(at 105.2 121.78 0)
+		(layer "F.SilkS")
+		(effects
+			(font
+				(size 0.6 0.6)
+				(thickness 0.09)
+			)
+			(justify left)
+		)
+	)
 	(gr_text "5V"
 		(at 120.44 104 0)
@@
 	)
 	(segment
-		(start 104 114.16)
-		(end 106.2 114.16)
-		(width 0.25)
-		(layer "F.Cu")
-		(net 5)
-	)
-	(segment
-		(start 106.2 114.16)
+		(start 104 116.7)
+		(end 106.2 116.7)
+		(width 0.25)
+		(layer "F.Cu")
+		(net 6)
+	)
+	(segment
+		(start 106.2 116.7)
 		(end 106.2 127)
 		(width 0.25)
 		(layer "F.Cu")
-		(net 5)
+		(net 6)
 	)
 	(segment
@@
 		(width 0.25)
 		(layer "F.Cu")
-		(net 5)
+		(net 6)
 	)
 	(segment
@@
 		(width 0.25)
 		(layer "F.Cu")
-		(net 5)
-	)
-	(segment
-		(start 104 116.7)
-		(end 105.7 116.7)
-		(width 0.25)
-		(layer "F.Cu")
 		(net 6)
 	)
 	(segment
-		(start 105.7 116.7)
+		(start 104 119.24)
+		(end 105.7 119.24)
+		(width 0.25)
+		(layer "F.Cu")
+		(net 7)
+	)
+	(segment
+		(start 105.7 119.24)
 		(end 105.7 127.5)
 		(width 0.25)
 		(layer "F.Cu")
-		(net 6)
+		(net 7)
 	)
 	(segment
@@
 		(width 0.25)
 		(layer "F.Cu")
-		(net 6)
+		(net 7)
 	)
 	(segment
@@
 		(width 0.25)
 		(layer "F.Cu")
-		(net 6)
+		(net 7)
+	)
+	(segment
+		(start 104 121.78)
+		(end 105.2 121.78)
+		(width 0.25)
+		(layer "F.Cu")
+		(net 8)
+	)
+	(segment
+		(start 105.2 121.78)
+		(end 105.2 128)
+		(width 0.25)
+		(layer "F.Cu")
+		(net 8)
+	)
+	(segment
+		(start 105.2 128)
+		(end 106.35 128)
+		(width 0.25)
+		(layer "F.Cu")
+		(net 8)
+	)
+	(segment
+		(start 106.35 128)
+		(end 106.35 132)
+		(width 0.25)
+		(layer "F.Cu")
+		(net 8)
 	)
 	(segment
@@
 		(layer "F.Cu")
 		(net 1)
-	)
-	(segment
-		(start 104 111.62)
-		(end 106.35 111.62)
-		(width 0.25)
-		(layer "B.Cu")
-		(net 4)
-	)
-	(segment
-		(start 106.35 111.62)
-		(end 106.35 129.4)
-		(width 0.25)
-		(layer "B.Cu")
-		(net 4)
-	)
-	(segment
-		(start 106.35 129.4)
-		(end 106.35 132)
-		(width 0.25)
-		(layer "F.Cu")
-		(net 4)
 	)
 	(segment
@@
 	)
 	(via
-		(at 106.35 129.4)
-		(size 0.8)
-		(drill 0.4)
-		(layers "F.Cu" "B.Cu")
-		(net 4)
-	)
-	(via
